File: Schematics/F20_Logic_Diagrams/F20_ROOT/F20_RIM.sch (KiCad schematic (older format))
At the start: 2 parts, among them U24 RIM

Commit message: 02/19/20 update
Connections:
- net LO_TIRE_TEMP: now reaches U24.A1
- net DD_RST: now reaches U24.A12
- net LC_TIRE_TEMP: now reaches U24.A2
- net LI_TIRE_TEMP: now reaches U24.A3
- net RO_TIRE_TEMP: now reaches U24.A4
- net RC_TIRE_TEMP: now reaches U24.A5
- net RI_TIRE_TEMP: now reaches U24.A6
- net RIM_RX3 renamed DD_TX
- net RIM_TX3 renamed DD_RX
Other:
- note added: "+5V Power Consumption\n 18mA for Tire Temp Sensors"
- note added: "LO : Left Outer\nLC : Left Center\nLI : Left Inner\nRO : Right Outer\nRC : Right Center\nRI : Right Inner"
Changed lines of the file:
@@
 $Descr A 11000 8500
 encoding utf-8
-Sheet 12 13
+Sheet 13 13
 Title "RIM"
 Date "2020-02-18"
@@
 Text GLabel 3500 4500 0    50   BiDi ~ 0
 RIM_SDA
-Text GLabel 3500 5000 0    50   BiDi ~ 0
-RIM_RX3
+Text GLabel 7500 5000 2    50   BiDi ~ 0
+DD_RX
 Wire Wire Line
 	3500 5000 5000 5000
@@
 Wire Wire Line
 	3500 2500 5000 2500
-Text GLabel 7500 5000 2    50   BiDi ~ 0
-RIM_TX3
+Text GLabel 3500 5000 0    50   BiDi ~ 0
+DD_TX
 Wire Wire Line
 	7500 5000 6000 5000
@@
 Wire Wire Line
 	2000 3500 2500 3500
+Text GLabel 7500 4750 2    50   Output ~ 0
+DD_RST
+Wire Wire Line
+	7500 2000 6000 2000
+Wire Wire Line
+	7500 4750 6000 4750
+Wire Wire Line
+	6000 2250 7500 2250
+Wire Wire Line
+	6000 2500 7500 2500
+Wire Wire Line
+	6000 2750 7500 2750
+Wire Wire Line
+	6000 3000 7500 3000
+Wire Wire Line
+	6000 3250 7500 3250
+Text GLabel 7500 2500 2    50   Input ~ 0
+LI_TIRE_TEMP
+Text GLabel 7500 2750 2    50   Input ~ 0
+RO_TIRE_TEMP
+Text GLabel 7500 3000 2    50   Input ~ 0
+RC_TIRE_TEMP
+Text GLabel 7500 3250 2    50   Input ~ 0
+RI_TIRE_TEMP
+Text Notes 5550 7550 0    50   ~ 0
+LO : Left Outer\nLC : Left Center\nLI : Left Inner\nRO : Right Outer\nRC : Right Center\nRI : Right Inner
+Wire Notes Line
+	5500 7000 5500 7600
+Text GLabel 7500 2000 2    50   Input ~ 0
+LO_TIRE_TEMP
+Text GLabel 7500 2250 2    50   Input ~ 0
+LC_TIRE_TEMP
+Text Notes 4250 7200 0    50   ~ 0
++5V Power Consumption\n   18mA for Tire Temp Sensors
+Wire Notes Line
+	4250 7000 4250 7600
+Wire Notes Line
+	4250 7600 6250 7600
+Wire Notes Line
+	4250 7000 6250 7000
 $EndSCHEMATC
