File: Schematics/F20_Logic_Diagrams/F20_ROOT/F20_RIM.sch (KiCad schematic (older format))
At the start: 2 parts, among them U24 RIM

Commit message: Added steering wheel drawing, udpated some ECU pinout to match previous tune, added accel/XBEE drawing
Connections:
- net RIM_AGND: now reaches U24.9 (AGND)
- net RIM_CANH renamed CANH
- net RIM_CANL renamed CANL
- net RIM_RX1 renamed XBEE_TX
- net RIM_TX1 renamed XBEE_RX
Changed lines of the file:
@@
 EESchema Schematic File Version 4
+LIBS:F20_ROOT-cache
 EELAYER 30 0
 EELAYER END
 $Descr A 11000 8500
 encoding utf-8
-Sheet 13 15
+Sheet 14 18
 Title "RIM"
 Date "2020-02-18"
@@
 	1    0    0    -1
 $EndComp
-Text GLabel 3500 2500 0    50   BiDi ~ 0
-RIM_CANH
-Text GLabel 3500 2750 0    50   BiDi ~ 0
-RIM_CANL
 Text GLabel 3500 3000 0    50   BiDi ~ 0
-RIM_RX1
+XBEE_TX
 Text GLabel 3500 3250 0    50   BiDi ~ 0
-RIM_TX1
+XBEE_RX
 Text GLabel 3500 3750 0    50   Output ~ 0
 RIM_+5V
@@
 Wire Notes Line
 	4250 7000 6250 7000
+Text GLabel 3500 2500 0    50   BiDi ~ 0
+CANH
+Text GLabel 3500 2750 0    50   BiDi ~ 0
+CANL
+Text GLabel 3500 4000 0    50   Output ~ 0
+RIM_AGND
+Wire Wire Line
+	3500 4000 5000 4000
 $EndSCHEMATC
