File: Schematics/F20_Logic_Diagrams/F20_ROOT/F20_Coils.sch (KiCad schematic (older format))
At the start: 1 part

Commit message: 02/18/20 update
Parts:
- gave numbers to parts that had none: 1
Changed lines of the file:
@@
 $Descr A 11000 8500
 encoding utf-8
-Sheet 5 11
+Sheet 5 13
 Title "Coil"
 Date "2020-02-04"
@@
 $EndDescr
 $Comp
-L FSAE_Library:Coil_Driver U?
+L FSAE_Library:Coil_Driver U4
 U 1 1 5E3A29CE
 P 4500 3000
-F 0 "U?" H 5250 3173 50  0000 C CNN
+F 0 "U4" H 5250 3173 50  0000 C CNN
 F 1 "Coil_Driver" H 4800 3150 50  0001 C CNN
 F 2 "" H 4800 3150 50  0001 C CNN
@@
 	8000 4000 6000 4000
 $Comp
-L FSAE_Library:GND_BAT #PWR?
+L FSAE_Library:GND_BAT #PWR04
 U 1 1 5E3A4419
 P 9000 4000
-F 0 "#PWR?" H 9000 3750 50  0001 C CNN
+F 0 "#PWR04" H 9000 3750 50  0001 C CNN
 F 1 "GND_BAT" H 9005 3827 50  0000 C CNN
 F 2 "" H 9000 4000 50  0001 C CNN

Commit message: 02/19/20 update
Parts:
- added U? (x4): Ignition_Coil, symbol FSAE_Library:Ignition_Coil
Connections:
- net Coil2 is gone; now on net GND: U4.3 (Coil2_Neg_Terminal)
- net Coil3 is gone; now on net COIL2_CTRL: U4.2 (ECU_Coil2_Output)
- net Coil3_CTRL is gone; now on net COIL3_CTRL: U4.4 (ECU_Coil3_Output)
- net Coil4 is gone; now on net COIL1_CTRL: U4.1 (ECU_Coil1_Output)
- net Coil1 renamed COIL3_CTRL
- net Coil1_CTRL renamed COIL1_CTRL
- net Coil2_CTRL renamed COIL2_CTRL
- net Coil4_CTRL renamed COIL4_CTRL
- new net: U4.1 (ECU_Coil1_Output), U?.2 (GND)
- new net: U4.2 (ECU_Coil2_Output), U?.2 (GND)
- new net: U4.3 (Coil2_Neg_Terminal), U?.2 (GND)
- new net: U4.4 (ECU_Coil3_Output), U?.2 (GND)
- new net COILS_PWR: U?.1 (+12V), U?.1 (+12V), U?.1 (+12V), U?.1 (+12V)
Changed lines of the file:
@@
 $EndComp
 Text GLabel 8000 3000 2    50   Input ~ 0
-Coil1_CTRL
+COIL1_CTRL
 Text GLabel 8000 3750 2    50   Input ~ 0
-Coil3_CTRL
+COIL3_CTRL
 Text GLabel 8000 4000 2    50   Input ~ 0
-Coil4_CTRL
+COIL4_CTRL
 Text GLabel 8000 3250 2    50   Input ~ 0
-Coil2_CTRL
+COIL2_CTRL
 Wire Wire Line
 	6000 3000 8000 3000
@@
 Wire Wire Line
 	9000 3500 6000 3500
-Text GLabel 2500 3000 0    50   Output ~ 0
-Coil1
-Text GLabel 2500 3250 0    50   Output ~ 0
-Coil2
-Text GLabel 2500 3500 0    50   Output ~ 0
-Coil3
-Text GLabel 2500 3750 0    50   Output ~ 0
-Coil4
 Wire Wire Line
-	2500 3000 4500 3000
+	3750 3000 4500 3000
 Wire Wire Line
-	4500 3250 2500 3250
+	4500 3250 3750 3250
 Wire Wire Line
-	2500 3500 4500 3500
+	3750 3500 4500 3500
 Wire Wire Line
-	4500 3750 2500 3750
+	4500 3750 3750 3750
+$Comp
+L FSAE_Library:Ignition_Coil U?
+U 1 1 5E52DBCE
+P 3000 3000
+F 0 "U?" H 3625 3125 50  0000 C CNN
+F 1 "Ignition_Coil" H 3300 3150 50  0001 C CNN
+F 2 "" H 3300 3150 50  0001 C CNN
+F 3 "" H 3300 3150 50  0001 C CNN
+F 4 "" H 3000 3000 50  0001 C CNN "PN"
+	1    3000 3000
+	1    0    0    -1
+$EndComp
+$Comp
+L FSAE_Library:Ignition_Coil U?
+U 1 1 5E5316CE
+P 3000 3250
+F 0 "U?" H 3625 3375 50  0000 C CNN
+F 1 "Ignition_Coil" H 3300 3400 50  0001 C CNN
+F 2 "" H 3300 3400 50  0001 C CNN
+F 3 "" H 3300 3400 50  0001 C CNN
+F 4 "" H 3000 3250 50  0001 C CNN "PN"
+	1    3000 3250
+	1    0    0    -1
+$EndComp
+$Comp
+L FSAE_Library:Ignition_Coil U?
+U 1 1 5E531907
+P 3000 3500
+F 0 "U?" H 3625 3625 50  0000 C CNN
+F 1 "Ignition_Coil" H 3300 3650 50  0001 C CNN
+F 2 "" H 3300 3650 50  0001 C CNN
+F 3 "" H 3300 3650 50  0001 C CNN
+F 4 "" H 3000 3500 50  0001 C CNN "PN"
+	1    3000 3500
+	1    0    0    -1
+$EndComp
+$Comp
+L FSAE_Library:Ignition_Coil U?
+U 1 1 5E531AD8
+P 3000 3750
+F 0 "U?" H 3625 3875 50  0000 C CNN
+F 1 "Ignition_Coil" H 3300 3900 50  0001 C CNN
+F 2 "" H 3300 3900 50  0001 C CNN
+F 3 "" H 3300 3900 50  0001 C CNN
+F 4 "" H 3000 3750 50  0001 C CNN "PN"
+	1    3000 3750
+	1    0    0    -1
+$EndComp
+Wire Wire Line
+	3000 3250 2500 3250
+Wire Wire Line
+	2500 3250 2500 3000
+Wire Wire Line
+	2500 3000 3000 3000
+Wire Wire Line
+	3000 3500 2500 3500
+Wire Wire Line
+	2500 3500 2500 3250
+Connection ~ 2500 3250
+Wire Wire Line
+	3000 3750 2500 3750
+Wire Wire Line
+	2500 3750 2500 3500
+Connection ~ 2500 3500
+Wire Wire Line
+	2500 3000 2000 3000
+Connection ~ 2500 3000
+Text GLabel 2000 3000 0    50   Input ~ 0
+COILS_PWR
 $EndSCHEMATC

Commit message: Update
Other:
- note added: "25mA max source current per coil\n100mA total"
Changed lines of the file:
@@
 EESchema Schematic File Version 4
-LIBS:F20_ROOT-cache
 EELAYER 30 0
 EELAYER END
@@
 Text GLabel 2000 3000 0    50   Input ~ 0
 COILS_PWR
+Text Notes 4900 7200 0    50   ~ 0
+25mA max source current per coil\n100mA total
 $EndSCHEMATC
