File: Schematics/F20_Logic_Diagrams/F20_ROOT/F20_Coils.sch (KiCad schematic (older format))
At the start: 5 parts, among them U4 Coil_Driver

Commit message: Re-annotated Logic Diagrams, pulled a BOM list based on Logic Diagrams
Parts:
- gave numbers to parts that had none: 4
- renumbered U4 to U24
Changed lines of the file:
@@
 $EndDescr
 $Comp
-L FSAE_Library:Coil_Driver U4
+L FSAE_Library:Coil_Driver U24
 U 1 1 5E3A29CE
 P 4500 3000
-F 0 "U4" H 5250 3173 50  0000 C CNN
+F 0 "U24" H 5250 3173 50  0000 C CNN
 F 1 "Coil_Driver" H 4800 3150 50  0001 C CNN
 F 2 "" H 4800 3150 50  0001 C CNN
@@
 	8000 4000 6000 4000
 $Comp
-L FSAE_Library:GND_BAT #PWR04
+L FSAE_Library:GND_BAT #PWR015
 U 1 1 5E3A4419
 P 9000 4000
-F 0 "#PWR04" H 9000 3750 50  0001 C CNN
+F 0 "#PWR015" H 9000 3750 50  0001 C CNN
 F 1 "GND_BAT" H 9005 3827 50  0000 C CNN
 F 2 "" H 9000 4000 50  0001 C CNN
@@
 	4500 3750 3750 3750
 $Comp
-L FSAE_Library:Ignition_Coil U?
+L FSAE_Library:Ignition_Coil U20
 U 1 1 5E52DBCE
 P 3000 3000
-F 0 "U?" H 3625 3125 50  0000 C CNN
+F 0 "U20" H 3625 3125 50  0000 C CNN
 F 1 "Ignition_Coil" H 3300 3150 50  0001 C CNN
 F 2 "" H 3300 3150 50  0001 C CNN
@@
 $EndComp
 $Comp
-L FSAE_Library:Ignition_Coil U?
+L FSAE_Library:Ignition_Coil U21
 U 1 1 5E5316CE
 P 3000 3250
-F 0 "U?" H 3625 3375 50  0000 C CNN
+F 0 "U21" H 3625 3375 50  0000 C CNN
 F 1 "Ignition_Coil" H 3300 3400 50  0001 C CNN
 F 2 "" H 3300 3400 50  0001 C CNN
@@
 $EndComp
 $Comp
-L FSAE_Library:Ignition_Coil U?
+L FSAE_Library:Ignition_Coil U22
 U 1 1 5E531907
 P 3000 3500
-F 0 "U?" H 3625 3625 50  0000 C CNN
+F 0 "U22" H 3625 3625 50  0000 C CNN
 F 1 "Ignition_Coil" H 3300 3650 50  0001 C CNN
 F 2 "" H 3300 3650 50  0001 C CNN
@@
 $EndComp
 $Comp
-L FSAE_Library:Ignition_Coil U?
+L FSAE_Library:Ignition_Coil U23
 U 1 1 5E531AD8
 P 3000 3750
-F 0 "U?" H 3625 3875 50  0000 C CNN
+F 0 "U23" H 3625 3875 50  0000 C CNN
 F 1 "Ignition_Coil" H 3300 3900 50  0001 C CNN
 F 2 "" H 3300 3900 50  0001 C CNN
