File: Schematics/F20_Logic_Diagrams/F20_ROOT/F20_Injectors.sch (KiCad schematic (older format))
At the start: 4 parts

Commit message: Update
Other:
- note added: "3A continous max per injector\n12A total"
Changed lines of the file:
@@
 EESchema Schematic File Version 4
-LIBS:F20_ROOT-cache
 EELAYER 30 0
 EELAYER END
@@
 Wire Wire Line
 	5750 4500 8000 4500
+Text Notes 5000 7200 0    50   ~ 0
+3A continous max per injector\n12A total
+Wire Notes Line
+	6250 7000 4950 7000
+Wire Notes Line
+	4950 7000 4950 7500
+Wire Notes Line
+	4950 7500 6250 7500
 $EndSCHEMATC
