File: Schematics/F20_Logic_Diagrams/F20_ROOT/F20_Power_Management.sch (KiCad schematic (older format))
At the start: 9 parts

Commit message: Added GND and GND_CHASSIS symbols, updated relevant schematics. Restructured Powertrain hierarchy. Created ECU Connector symbols.
Connections:
- net labels added: GND_BAT
- wire segments 26 -> 28
Changed lines of the file:
@@
-	1    0    0    -1
-$EndComp
-$Comp
-L power:GND #PWR?
-U 1 1 5E234DD1
-P 3000 3500
-F 0 "#PWR?" H 3000 3250 50  0001 C CNN
-F 1 "GND" H 3005 3327 50  0000 C CNN
-F 2 "" H 3000 3500 50  0001 C CNN
-F 3 "" H 3000 3500 50  0001 C CNN
-	1    3000 3500
 	1    0    0    -1
 $EndComp
@@
 Wire Wire Line
 	4800 3250 5500 3250
-$Comp
-L power:GND #PWR?
-U 1 1 5E23A8FA
-P 4000 3500
-F 0 "#PWR?" H 4000 3250 50  0001 C CNN
-F 1 "GND" H 4005 3327 50  0000 C CNN
-F 2 "" H 4000 3500 50  0001 C CNN
-F 3 "" H 4000 3500 50  0001 C CNN
-	1    4000 3500
-	1    0    0    -1
-$EndComp
 Wire Wire Line
 	4000 3500 4000 3250
@@
 Wire Wire Line
 	5000 4750 4750 4750
-$Comp
-L power:GND #PWR?
-U 1 1 5E2174D8
-P 5000 5000
-F 0 "#PWR?" H 5000 4750 50  0001 C CNN
-F 1 "GND" H 5005 4827 50  0000 C CNN
-F 2 "" H 5000 5000 50  0001 C CNN
-F 3 "" H 5000 5000 50  0001 C CNN
-	1    5000 5000
-	-1   0    0    -1
-$EndComp
 Wire Wire Line
 	4000 4500 3500 4500
@@
 Wire Wire Line
 	6250 4500 6500 4500
-$Comp
-L power:GND #PWR?
-U 1 1 5E330233
-P 7250 4700
-F 0 "#PWR?" H 7250 4450 50  0001 C CNN
-F 1 "GND" H 7255 4527 50  0000 C CNN
-F 2 "" H 7250 4700 50  0001 C CNN
-F 3 "" H 7250 4700 50  0001 C CNN
-	1    7250 4700
-	-1   0    0    -1
-$EndComp
 Wire Wire Line
 	6500 3250 6500 4000
@@
 Text Notes 7500 4550 0    50   ~ 0
 IGN SW input to ECU?
+$Comp
+L FSAE_Library:GND #PWR?
+U 1 1 5E3B4E50
+P 4000 3500
+F 0 "#PWR?" H 4000 3300 50  0001 C CNN
+F 1 "GND" H 4004 3346 50  0000 C CNN
+F 2 "" H 4000 3450 50  0001 C CNN
+F 3 "" H 4000 3450 50  0001 C CNN
+	1    4000 3500
+	1    0    0    -1
+$EndComp
+$Comp
+L FSAE_Library:GND #PWR?
+U 1 1 5E3B6858
+P 5000 5000
+F 0 "#PWR?" H 5000 4800 50  0001 C CNN
+F 1 "GND" H 5004 4846 50  0000 C CNN
+F 2 "" H 5000 4950 50  0001 C CNN
+F 3 "" H 5000 4950 50  0001 C CNN
+	1    5000 5000
+	1    0    0    -1
+$EndComp
+$Comp
+L FSAE_Library:GND #PWR?
+U 1 1 5E3B6F4B
+P 7250 4700
+F 0 "#PWR?" H 7250 4500 50  0001 C CNN
+F 1 "GND" H 7254 4546 50  0000 C CNN
+F 2 "" H 7250 4650 50  0001 C CNN
+F 3 "" H 7250 4650 50  0001 C CNN
+	1    7250 4700
+	1    0    0    -1
+$EndComp
+$Comp
+L FSAE_Library:GND #PWR?
+U 1 1 5E3B7E28
+P 3000 3500
+F 0 "#PWR?" H 3000 3300 50  0001 C CNN
+F 1 "GND" H 3004 3346 50  0000 C CNN
+F 2 "" H 3000 3450 50  0001 C CNN
+F 3 "" H 3000 3450 50  0001 C CNN
+	1    3000 3500
+	1    0    0    -1
+$EndComp
+$Comp
+L FSAE_Library:GND_BAT #PWR?
+U 1 1 5E3B8350
+P 2500 3500
+F 0 "#PWR?" H 2500 3250 50  0001 C CNN
+F 1 "GND_BAT" H 2505 3327 50  0000 C CNN
+F 2 "" H 2500 3500 50  0001 C CNN
+F 3 "" H 2500 3500 50  0001 C CNN
+	1    2500 3500
+	1    0    0    -1
+$EndComp
+Wire Wire Line
+	2500 3500 2500 3000
+Wire Wire Line
+	2500 3000 3000 3000
+Connection ~ 3000 3000
 $EndSCHEMATC

Commit message: Updated per AD commit. O2 sensor schematic, transponder schematic.
Connections:
- new net: S?.~, U?.~ (Start)
Changed lines of the file:
@@
 EESchema Schematic File Version 4
-LIBS:F20_ROOT-cache
 EELAYER 30 0
 EELAYER END
 $Descr A 11000 8500
 encoding utf-8
-Sheet 6 7
+Sheet 6 9
 Title "Fuses and Relays"
 Date "2020-01-28"

Commit message: Weekly update. Added Tire temp sensors drawing.
Connections:
- new net: S?.~, U?.~ (Start)
Changed lines of the file:
@@
 EESchema Schematic File Version 4
+LIBS:F20_ROOT-cache
 EELAYER 30 0
 EELAYER END
 $Descr A 11000 8500
 encoding utf-8
-Sheet 6 9
+Sheet 8 11
 Title "Fuses and Relays"
 Date "2020-01-28"
@@
 IGN SW input to ECU?
 $Comp
-L FSAE_Library:GND #PWR?
+L FSAE_Library:GND #PWR0106
 U 1 1 5E3B4E50
 P 4000 3500
-F 0 "#PWR?" H 4000 3300 50  0001 C CNN
+F 0 "#PWR0106" H 4000 3300 50  0001 C CNN
 F 1 "GND" H 4004 3346 50  0000 C CNN
 F 2 "" H 4000 3450 50  0001 C CNN
@@
 $EndComp
 $Comp
-L FSAE_Library:GND #PWR?
+L FSAE_Library:GND #PWR0107
 U 1 1 5E3B6858
 P 5000 5000
-F 0 "#PWR?" H 5000 4800 50  0001 C CNN
+F 0 "#PWR0107" H 5000 4800 50  0001 C CNN
 F 1 "GND" H 5004 4846 50  0000 C CNN
 F 2 "" H 5000 4950 50  0001 C CNN
@@
 $EndComp
 $Comp
-L FSAE_Library:GND #PWR?
+L FSAE_Library:GND #PWR0108
 U 1 1 5E3B6F4B
 P 7250 4700
-F 0 "#PWR?" H 7250 4500 50  0001 C CNN
+F 0 "#PWR0108" H 7250 4500 50  0001 C CNN
 F 1 "GND" H 7254 4546 50  0000 C CNN
 F 2 "" H 7250 4650 50  0001 C CNN
@@
 $EndComp
 $Comp
-L FSAE_Library:GND #PWR?
+L FSAE_Library:GND #PWR0109
 U 1 1 5E3B7E28
 P 3000 3500
-F 0 "#PWR?" H 3000 3300 50  0001 C CNN
+F 0 "#PWR0109" H 3000 3300 50  0001 C CNN
 F 1 "GND" H 3004 3346 50  0000 C CNN
 F 2 "" H 3000 3450 50  0001 C CNN
@@
 $EndComp
 $Comp
-L FSAE_Library:GND_BAT #PWR?
+L FSAE_Library:GND_BAT #PWR0110
 U 1 1 5E3B8350
 P 2500 3500
-F 0 "#PWR?" H 2500 3250 50  0001 C CNN
+F 0 "#PWR0110" H 2500 3250 50  0001 C CNN
 F 1 "GND_BAT" H 2505 3327 50  0000 C CNN
 F 2 "" H 2500 3500 50  0001 C CNN

Commit message: 02/18/20 update
Parts:
- R1: renamed from R?; value 3 -> 3Ω
- gave numbers to parts that had none: 8
Connections:
- new net: S1.~, U15.~ (Start)
Changed lines of the file:
@@
 $Descr A 11000 8500
 encoding utf-8
-Sheet 8 11
+Sheet 9 13
 Title "Fuses and Relays"
 Date "2020-01-28"
@@
 BAT_PWR
 $Comp
-L FSAE_Library:Battery U?
+L FSAE_Library:Battery U11
 U 1 1 5E233AF7
 P 4000 3000
-F 0 "U?" H 3750 3173 50  0000 C CNN
+F 0 "U11" H 3750 3173 50  0000 C CNN
 F 1 "Battery" H 3750 3150 50  0001 C CNN
 F 2 "" H 3750 3150 50  0001 C CNN
@@
 	3000 3000 3500 3000
 $Comp
-L FSAE_Library:Cutoff_Switch U?
+L FSAE_Library:Cutoff_Switch U12
 U 1 1 5E237569
 P 5500 3000
-F 0 "U?" H 5875 3173 50  0000 C CNN
+F 0 "U12" H 5875 3173 50  0000 C CNN
 F 1 "Cutoff_Switch" H 5850 3150 50  0001 C CNN
 F 2 "" H 5850 3150 50  0001 C CNN
@@
 	4000 3250 4500 3250
 $Comp
-L Device:R_US R?
+L Device:R_US R1
 U 1 1 5E2398AB
 P 4650 3250
-F 0 "R?" V 4550 3250 50  0000 C CNN
-F 1 "3" V 4750 3250 50  0000 C CNN
+F 0 "R1" V 4550 3250 50  0000 C CNN
+F 1 "3Ω" V 4750 3250 50  0000 C CNN
 F 2 "" V 4690 3240 50  0001 C CNN
 F 3 "~" H 4650 3250 50  0001 C CNN
@@
 	5000 3000 5500 3000
 $Comp
-L FSAE_Library:Fuse F?
+L FSAE_Library:Fuse F1
 U 1 1 5E24B48F
 P 4700 3000
-F 0 "F?" H 4850 3100 50  0000 C CNN
+F 0 "F1" H 4850 3100 50  0000 C CNN
 F 1 "100A" H 4850 2900 50  0000 C CNN
 F 2 "" H 4850 3080 50  0001 C CNN
@@
 	4000 4000 3500 4000
 $Comp
-L FSAE_Library:Alternator U?
+L FSAE_Library:Alternator U13
 U 1 1 5E21541A
 P 3500 4000
-F 0 "U?" H 3750 4150 50  0000 L CNN
+F 0 "U13" H 3750 4150 50  0000 L CNN
 F 1 "Alternator" H 3800 4150 50  0001 C CNN
 F 2 "" H 3800 4150 50  0001 C CNN
@@
 $EndComp
 $Comp
-L FSAE_Library:Rectifier U?
+L FSAE_Library:Rectifier U14
 U 1 1 5E21334A
 P 4750 4000
-F 0 "U?" H 5150 4150 50  0000 C CNN
+F 0 "U14" H 5150 4150 50  0000 C CNN
 F 1 "Rectifier" H 5000 4150 50  0001 C CNN
 F 2 "" H 5250 4500 50  0001 C CNN
@@
 $EndComp
 $Comp
-L FSAE_Library:Starter_Relay U?
+L FSAE_Library:Starter_Relay U15
 U 1 1 5E3285A1
 P 5500 4000
-F 0 "U?" H 5875 4173 50  0000 C CNN
+F 0 "U15" H 5875 4173 50  0000 C CNN
 F 1 "Starter_Relay" H 5750 4150 50  0001 C CNN
 F 2 "" H 6000 4500 50  0001 C CNN
@@
 Connection ~ 6500 3250
 $Comp
-L FSAE_Library:Starter_Motor U?
+L FSAE_Library:Starter_Motor U16
 U 1 1 5E3347A8
 P 6500 4250
-F 0 "U?" H 6700 4400 50  0000 L CNN
+F 0 "U16" H 6700 4400 50  0000 L CNN
 F 1 "Starter_Motor" H 6750 4400 50  0001 C CNN
 F 2 "" H 6750 4400 50  0001 C CNN
@@
 	6500 4250 6250 4250
 $Comp
-L FSAE_Library:Ignition_SW S?
+L FSAE_Library:Ignition_SW S1
 U 1 1 5E335D97
 P 6500 4500
-F 0 "S?" H 6750 4600 50  0000 C CNN
+F 0 "S1" H 6750 4600 50  0000 C CNN
 F 1 "Ignition_SW" H 6575 4650 50  0001 L CNN
 F 2 "" H 6600 4200 50  0001 L CNN
@@
 IGN SW input to ECU?
 $Comp
-L FSAE_Library:GND #PWR0106
+L FSAE_Library:GND #PWR011
 U 1 1 5E3B4E50
 P 4000 3500
-F 0 "#PWR0106" H 4000 3300 50  0001 C CNN
+F 0 "#PWR011" H 4000 3300 50  0001 C CNN
 F 1 "GND" H 4004 3346 50  0000 C CNN
 F 2 "" H 4000 3450 50  0001 C CNN
@@
 $EndComp
 $Comp
-L FSAE_Library:GND #PWR0107
+L FSAE_Library:GND #PWR013
 U 1 1 5E3B6858
 P 5000 5000
-F 0 "#PWR0107" H 5000 4800 50  0001 C CNN
+F 0 "#PWR013" H 5000 4800 50  0001 C CNN
 F 1 "GND" H 5004 4846 50  0000 C CNN
 F 2 "" H 5000 4950 50  0001 C CNN
@@
 $EndComp
 $Comp
-L FSAE_Library:GND #PWR0108
+L FSAE_Library:GND #PWR012
 U 1 1 5E3B6F4B
 P 7250 4700
-F 0 "#PWR0108" H 7250 4500 50  0001 C CNN
+F 0 "#PWR012" H 7250 4500 50  0001 C CNN
 F 1 "GND" H 7254 4546 50  0000 C CNN
 F 2 "" H 7250 4650 50  0001 C CNN
@@
 $EndComp
 $Comp
-L FSAE_Library:GND #PWR0109
+L FSAE_Library:GND #PWR010
 U 1 1 5E3B7E28
 P 3000 3500
-F 0 "#PWR0109" H 3000 3300 50  0001 C CNN
+F 0 "#PWR010" H 3000 3300 50  0001 C CNN
 F 1 "GND" H 3004 3346 50  0000 C CNN
 F 2 "" H 3000 3450 50  0001 C CNN
@@
 $EndComp
 $Comp
-L FSAE_Library:GND_BAT #PWR0110
+L FSAE_Library:GND_BAT #PWR09
 U 1 1 5E3B8350
 P 2500 3500
-F 0 "#PWR0110" H 2500 3250 50  0001 C CNN
+F 0 "#PWR09" H 2500 3250 50  0001 C CNN
 F 1 "GND_BAT" H 2505 3327 50  0000 C CNN
 F 2 "" H 2500 3500 50  0001 C CNN

Commit message: Added injectors drawing
Connections:
- new net: S1.~, U15.~ (Start)
Changed lines of the file:
@@
 $Descr A 11000 8500
 encoding utf-8
-Sheet 9 13
+Sheet 9 14
 Title "Fuses and Relays"
 Date "2020-01-28"

Commit message: Major powertrain update, added shifting schematic
Connections:
- new net: S1.~, U15.~ (Start)
Changed lines of the file:
@@
 $Descr A 11000 8500
 encoding utf-8
-Sheet 9 14
+Sheet 10 15
 Title "Fuses and Relays"
 Date "2020-01-28"

Commit message: Update
Connections:
- new net: S1.~, U15.~ (Start)
Changed lines of the file:
@@
 EESchema Schematic File Version 4
-LIBS:F20_ROOT-cache
 EELAYER 30 0
 EELAYER END

Commit message: Added steering wheel drawing, udpated some ECU pinout to match previous tune, added accel/XBEE drawing
Connections:
- new net: S1.~, U15.~ (Start)
Changed lines of the file:
@@
 EESchema Schematic File Version 4
+LIBS:F20_ROOT-cache
 EELAYER 30 0
 EELAYER END
 $Descr A 11000 8500
 encoding utf-8
-Sheet 10 15
+Sheet 10 18
 Title "Fuses and Relays"
 Date "2020-01-28"
@@
 U 1 1 5E21541A
 P 3500 4000
+AR Path="/5E21541A" Ref="U13"  Part="1"
+AR Path="/5E1D1A8A/5E21541A" Ref="U13"  Part="1"
 F 0 "U13" H 3750 4150 50  0000 L CNN
 F 1 "Alternator" H 3800 4150 50  0001 C CNN
