File: Schematics/F20_Logic_Diagrams/F20_ROOT/F20_ROOT.sch (KiCad schematic (older format))
At the start: 0 parts

Commit message: Major powertrain update, added shifting schematic
Changed lines of the file:
@@
 $Descr A4 11693 8268
 encoding utf-8
-Sheet 1 14
+Sheet 1 15
 Title "Root Index"
 Date ""
@@
 F1 "F20_RIM.sch" 50
 $EndSheet
+$Sheet
+S 3000 2000 1700 700
+U 5E6277A0
+F0 "Shifter" 50
+F1 "F20_Shifter.sch" 50
+$EndSheet
 $EndSCHEMATC

Commit message: Added steering wheel drawing, udpated some ECU pinout to match previous tune, added accel/XBEE drawing
Changed lines of the file:
@@
 EESchema Schematic File Version 4
+LIBS:F20_ROOT-cache
 EELAYER 30 0
 EELAYER END
 $Descr A4 11693 8268
 encoding utf-8
-Sheet 1 15
+Sheet 1 18
 Title "Root Index"
 Date ""
@@
 F1 "F20_Shifter.sch" 50
 $EndSheet
+$Sheet
+S 3000 3000 1700 700
+U 5E698156
+F0 "Steering Wheel" 50
+F1 "F20_Steering.sch" 50
+$EndSheet
+$Sheet
+S 3000 4000 1700 700
+U 5E6ABD2F
+F0 "XBEE" 50
+F1 "F20_XBEE.sch" 50
+$EndSheet
+$Sheet
+S 3000 5000 1700 700
+U 5E6AC2D1
+F0 "Accelerometer" 50
+F1 "F20_Accelerometer.sch" 50
+$EndSheet
 $EndSCHEMATC
