File: Schematics/F20_Logic_Diagrams/F20_ROOT/F20_Transponder.sch (KiCad schematic (older format))
At the start: 1 part

Commit message: 02/18/20 update
Parts:
- gave numbers to parts that had none: 1
Changed lines of the file:
@@
 $Descr A 11000 8500
 encoding utf-8
-Sheet 10 11
+Sheet 10 13
 Title "Transponder"
 Date "2020-02-03"
@@
 $EndDescr
 $Comp
-L FSAE_Library:Transponder U?
+L FSAE_Library:Transponder U17
 U 1 1 5E38FBDA
 P 7500 3500
-F 0 "U?" H 8028 3350 50  0000 L CNN
+F 0 "U17" H 8028 3350 50  0000 L CNN
 F 1 "Transponder" H 7650 3550 50  0001 C CNN
 F 2 "" H 8000 4000 50  0001 C CNN
@@
 	3000 3750 3000 4000
 $Comp
-L FSAE_Library:GND #PWR0112
+L FSAE_Library:GND #PWR015
 U 1 1 5E3B8D8B
 P 3000 4000
-F 0 "#PWR0112" H 3000 3800 50  0001 C CNN
+F 0 "#PWR015" H 3000 3800 50  0001 C CNN
 F 1 "GND" H 3004 3846 50  0000 C CNN
 F 2 "" H 3000 3950 50  0001 C CNN
