File: Schematics/F20_Logic_Diagrams/F20_ROOT/F20_Accelerometer.sch (KiCad schematic (older format))
At the start: 1 part

Commit message: Re-annotated Logic Diagrams, pulled a BOM list based on Logic Diagrams
Parts:
- gave numbers to parts that had none: 1
Changed lines of the file:
@@
 $EndDescr
 $Comp
-L FSAE_Library:BNO055 U?
+L FSAE_Library:BNO055 U48
 U 1 1 5E6DCC7F
 P 8000 3000
-F 0 "U?" H 8528 2600 50  0000 L CNN
+F 0 "U48" H 8528 2600 50  0000 L CNN
 F 1 "BNO055" H 8300 3250 50  0001 C CNN
 F 2 "" H 8500 3500 50  0001 C CNN
