File: Schematics/F20_Logic_Diagrams/F20_ROOT/F20_Driver_Display.sch (KiCad schematic (older format))
At the start: 1 part, among them U6 Driver_Display

Commit message: Re-annotated Logic Diagrams, pulled a BOM list based on Logic Diagrams
Parts:
- renumbered U6 to U29
Changed lines of the file:
@@
 $Descr A 11000 8500
 encoding utf-8
-Sheet 8 18
+Sheet 10 18
 Title "FSAE"
 Date "2020-02-03"
@@
 $EndDescr
 $Comp
-L FSAE_Library:Driver_Display U6
+L FSAE_Library:Driver_Display U29
 U 1 1 5E291EA2
 P 7500 3000
-F 0 "U6" H 7750 3150 50  0000 L CNN
+F 0 "U29" H 7750 3150 50  0000 L CNN
 F 1 "Driver_Display" H 7800 3150 50  0001 C CNN
 F 2 "" H 7800 3150 50  0001 C CNN
@@
 	4500 4000 7500 4000
 $Comp
-L FSAE_Library:GND #PWR07
+L FSAE_Library:GND #PWR016
 U 1 1 5E3C11D7
 P 3500 3500
-F 0 "#PWR07" H 3500 3300 50  0001 C CNN
+F 0 "#PWR016" H 3500 3300 50  0001 C CNN
 F 1 "GND" H 3504 3346 50  0000 C CNN
 F 2 "" H 3500 3450 50  0001 C CNN
