File: Schematics/F20_Logic_Diagrams/F20_ROOT/F20_ECU_CONN1.sch (KiCad schematic (older format))
At the start: 1 part, among them U2 ECU_Conn1

Commit message: Added PDM Layout guide, updated Powertrain wiring, added a Master Connector Pinout guide, added TOC to LogicDiagrams pdf and rearranged them a bit.
Other:
- note removed: "Shift up\nShift down\nClutch"
Changed lines of the file:
@@
 Wire Wire Line
 	2500 5650 4500 5650
-Text Notes 8150 2150 0    200  ~ 40
-Shift up\nShift down\nClutch
 Text Notes 1550 2250 0    50   ~ 0
 Connect to a harness

Commit message: Re-annotated Logic Diagrams, pulled a BOM list based on Logic Diagrams
Parts:
- renumbered U2 to U16
Changed lines of the file:
@@
 $EndDescr
 $Comp
-L FSAE_Library:ECU_Conn1 U2
+L FSAE_Library:ECU_Conn1 U16
 U 1 1 5E3C649A
 P 4500 1000
-F 0 "U2" H 5250 1173 50  0000 C CNN
+F 0 "U16" H 5250 1173 50  0000 C CNN
 F 1 "ECU_Conn1" H 5250 1150 50  0001 C CNN
 F 2 "" H 5000 2000 50  0001 C CNN
@@
 	2500 5200 4500 5200
 $Comp
-L FSAE_Library:GND_BAT #PWR02
+L FSAE_Library:GND_BAT #PWR010
 U 1 1 5E44A710
 P 6500 6450
-F 0 "#PWR02" H 6500 6200 50  0001 C CNN
+F 0 "#PWR010" H 6500 6200 50  0001 C CNN
 F 1 "GND_BAT" H 6505 6277 50  0000 C CNN
 F 2 "" H 6500 6450 50  0001 C CNN
@@
 	4000 5350 4000 6500
 $Comp
-L FSAE_Library:GND_BAT #PWR03
+L FSAE_Library:GND_BAT #PWR09
 U 1 1 5E4538FC
 P 4000 6500
-F 0 "#PWR03" H 4000 6250 50  0001 C CNN
+F 0 "#PWR09" H 4000 6250 50  0001 C CNN
 F 1 "GND_BAT" H 4005 6327 50  0000 C CNN
 F 2 "" H 4000 6500 50  0001 C CNN
