File: Schematics/F20_Logic_Diagrams/F20_ROOT/F20_Powertrain.sch (KiCad schematic (older format))
At the start: 9 parts, among them U1 Fan

Commit message: Re-annotated Logic Diagrams, pulled a BOM list based on Logic Diagrams
Parts:
- U12: renamed from U?; symbol FSAE_Library:Intake_Air_Temp -> FSAE_Library:IAT_Sensor
- U8: renamed from U?; symbol FSAE_Library:Throttle_Position_Sensor -> FSAE_Library:TP_Sensor
- gave numbers to parts that had none: 6
- renumbered U1 to U7
Changed lines of the file:
@@
 $EndSheet
 $Comp
-L FSAE_Library:Fan U1
+L FSAE_Library:Fan U7
 U 1 1 5E3D2712
 P 3500 1000
-F 0 "U1" H 3875 1173 50  0000 C CNN
+F 0 "U7" H 3875 1173 50  0000 C CNN
 F 1 "Fan" H 3750 1150 50  0001 C CNN
 F 2 "" H 4000 1500 50  0001 C CNN
@@
 $EndComp
 $Comp
-L FSAE_Library:GND #PWR01
+L FSAE_Library:GND #PWR07
 U 1 1 5E3D3AE8
 P 2000 1500
-F 0 "#PWR01" H 2000 1300 50  0001 C CNN
+F 0 "#PWR07" H 2000 1300 50  0001 C CNN
 F 1 "GND" H 2004 1346 50  0000 C CNN
 F 2 "" H 2000 1450 50  0001 C CNN
@@
 P 3500 5000
 AR Path="/5E5F0904/5E5FB918" Ref="U?"  Part="1"
-AR Path="/5E1D1B45/5E5FB918" Ref="U?"  Part="1"
-F 0 "U?" H 4028 4875 50  0000 L CNN
+AR Path="/5E1D1B45/5E5FB918" Ref="U10"  Part="1"
+F 0 "U10" H 4028 4875 50  0000 L CNN
 F 1 "Fuel_Pump" H 3750 5150 50  0001 C CNN
 F 2 "" H 4000 5500 50  0001 C CNN
@@
 P 2000 5500
 AR Path="/5E5F0904/5E5FB922" Ref="#PWR?"  Part="1"
-AR Path="/5E1D1B45/5E5FB922" Ref="#PWR?"  Part="1"
-F 0 "#PWR?" H 2000 5300 50  0001 C CNN
+AR Path="/5E1D1B45/5E5FB922" Ref="#PWR08"  Part="1"
+F 0 "#PWR08" H 2000 5300 50  0001 C CNN
 F 1 "GND" H 2004 5346 50  0000 C CNN
 F 2 "" H 2000 5450 50  0001 C CNN
@@
 $EndComp
 $Comp
-L FSAE_Library:Intake_Air_Temp U?
+L FSAE_Library:IAT_Sensor U?
 U 1 1 5E5FB938
 P 6500 1000
 AR Path="/5E5F0904/5E5FB938" Ref="U?"  Part="1"
-AR Path="/5E1D1B45/5E5FB938" Ref="U?"  Part="1"
-F 0 "U?" H 7028 875 50  0000 L CNN
+AR Path="/5E1D1B45/5E5FB938" Ref="U12"  Part="1"
+F 0 "U12" H 7028 875 50  0000 L CNN
 F 1 "Intake_Air_Temp" H 6750 1150 50  0001 C CNN
 F 2 "" H 7000 1500 50  0001 C CNN
@@
 IAT_SIG
 $Comp
-L FSAE_Library:Throttle_Position_Sensor U?
+L FSAE_Library:TP_Sensor U?
 U 1 1 5E5FB942
 P 3500 2000
 AR Path="/5E5F0904/5E5FB942" Ref="U?"  Part="1"
-AR Path="/5E1D1B45/5E5FB942" Ref="U?"  Part="1"
-F 0 "U?" H 4028 1725 50  0000 L CNN
+AR Path="/5E1D1B45/5E5FB942" Ref="U8"  Part="1"
+F 0 "U8" H 4028 1725 50  0000 L CNN
 F 1 "Throttle_Position_Sensor" H 3800 2150 50  0001 C CNN
 F 2 "" H 4000 2500 50  0001 C CNN
@@
 P 6500 2000
 AR Path="/5E5F0904/5E5FB94E" Ref="U?"  Part="1"
-AR Path="/5E1D1B45/5E5FB94E" Ref="U?"  Part="1"
-F 0 "U?" H 7028 1725 50  0000 L CNN
+AR Path="/5E1D1B45/5E5FB94E" Ref="U13"  Part="1"
+F 0 "U13" H 7028 1725 50  0000 L CNN
 F 1 "MAP_Sensor" H 6800 2150 50  0001 C CNN
 F 2 "" H 7000 2500 50  0001 C CNN
@@
 CAM_VR-
 $Comp
-L FSAE_Library:Camshaft_Sensor U?
+L FSAE_Library:Camshaft_Sensor U14
 U 1 1 5E665C35
 P 6500 3500
-F 0 "U?" H 7028 3250 50  0000 L CNN
+F 0 "U14" H 7028 3250 50  0000 L CNN
 F 1 "Camshaft_Sensor" H 6750 3650 50  0001 C CNN
 F 2 "" H 7000 4000 50  0001 C CNN
@@
 $EndComp
 $Comp
-L FSAE_Library:Crankshaft_Sensor U?
+L FSAE_Library:Crankshaft_Sensor U9
 U 1 1 5E6666BD
 P 3500 3500
-F 0 "U?" H 4028 3250 50  0000 L CNN
+F 0 "U9" H 4028 3250 50  0000 L CNN
 F 1 "Crankshaft_Sensor" H 3750 3650 50  0001 C CNN
 F 2 "" H 4000 4000 50  0001 C CNN
@@
 U 1 1 5E695F31
 P 6500 5000
-F 0 "U?" H 7028 4875 50  0000 L CNN
+AR Path="/5E695F31" Ref="U?"  Part="1"
+AR Path="/5E1D1B45/5E695F31" Ref="U15"  Part="1"
+F 0 "U15" H 7028 4875 50  0000 L CNN
 F 1 "ECT_Sensor" H 6750 5150 50  0001 C CNN
 F 2 "" H 7000 5500 50  0001 C CNN
@@
 $EndComp
 $Comp
-L FSAE_Library:EOP_Sensor U?
+L FSAE_Library:EOP_Sensor U11
 U 1 1 5E696BEC
 P 3500 6000
-F 0 "U?" H 4028 5725 50  0000 L CNN
+F 0 "U11" H 4028 5725 50  0000 L CNN
 F 1 "EOP_Sensor" H 3800 6150 50  0001 C CNN
 F 2 "" H 4000 6500 50  0001 C CNN
