File: Schematics/F20_Logic_Diagrams/F20_ROOT/F20_Tire_Temp_Sensors.sch (KiCad schematic (older format))
At the start: 6 parts, among them U18 Tire_Temp_Sensor, U19 Tire_Temp_Sensor, U20 Tire_Temp_Sensor, U21 Tire_Temp_Sensor, U22 Tire_Temp_Sensor, U23 Tire_Temp_Sensor

Commit message: Re-annotated Logic Diagrams, pulled a BOM list based on Logic Diagrams
Parts:
- renumbered U18 to U35, U19 to U36, U20 to U37, U21 to U38, U22 to U39, U23 to U40
Changed lines of the file:
@@
 $EndDescr
 $Comp
-L FSAE_Library:Tire_Temp_Sensor U18
+L FSAE_Library:Tire_Temp_Sensor U35
 U 1 1 5E3B80AD
 P 8500 1000
-F 0 "U18" H 9028 725 50  0000 L CNN
+F 0 "U35" H 9028 725 50  0000 L CNN
 F 1 "Tire_Temp_Sensor" H 8650 1050 50  0001 C CNN
 F 2 "" H 9000 1500 50  0001 C CNN
@@
 $EndComp
 $Comp
-L FSAE_Library:Tire_Temp_Sensor U19
+L FSAE_Library:Tire_Temp_Sensor U36
 U 1 1 5E3B9299
 P 8500 2000
-F 0 "U19" H 9028 1725 50  0000 L CNN
+F 0 "U36" H 9028 1725 50  0000 L CNN
 F 1 "Tire_Temp_Sensor" H 8650 2050 50  0001 C CNN
 F 2 "" H 9000 2500 50  0001 C CNN
@@
 $EndComp
 $Comp
-L FSAE_Library:Tire_Temp_Sensor U20
+L FSAE_Library:Tire_Temp_Sensor U37
 U 1 1 5E3BA080
 P 8500 3000
-F 0 "U20" H 9028 2725 50  0000 L CNN
+F 0 "U37" H 9028 2725 50  0000 L CNN
 F 1 "Tire_Temp_Sensor" H 8650 3050 50  0001 C CNN
 F 2 "" H 9000 3500 50  0001 C CNN
@@
 $EndComp
 $Comp
-L FSAE_Library:Tire_Temp_Sensor U21
+L FSAE_Library:Tire_Temp_Sensor U38
 U 1 1 5E3BAAB5
 P 8500 4000
-F 0 "U21" H 9028 3725 50  0000 L CNN
+F 0 "U38" H 9028 3725 50  0000 L CNN
 F 1 "Tire_Temp_Sensor" H 8650 4050 50  0001 C CNN
 F 2 "" H 9000 4500 50  0001 C CNN
@@
 	3500 2000 8500 2000
 $Comp
-L FSAE_Library:Tire_Temp_Sensor U22
+L FSAE_Library:Tire_Temp_Sensor U39
 U 1 1 5E3CA66D
 P 8500 5000
-F 0 "U22" H 9028 4725 50  0000 L CNN
+F 0 "U39" H 9028 4725 50  0000 L CNN
 F 1 "Tire_Temp_Sensor" H 8650 5050 50  0001 C CNN
 F 2 "" H 9000 5500 50  0001 C CNN
@@
 RIM_+5V
 $Comp
-L FSAE_Library:Tire_Temp_Sensor U23
+L FSAE_Library:Tire_Temp_Sensor U40
 U 1 1 5E3CFAE2
 P 8500 6000
-F 0 "U23" H 9028 5725 50  0000 L CNN
+F 0 "U40" H 9028 5725 50  0000 L CNN
 F 1 "Tire_Temp_Sensor" H 8650 6050 50  0001 C CNN
 F 2 "" H 9000 6500 50  0001 C CNN
