File: Schematics/F20_Logic_Diagrams/F20_ROOT/F20_XBEE.sch (KiCad schematic (older format))
At the start: 1 part

Commit message: Re-annotated Logic Diagrams, pulled a BOM list based on Logic Diagrams
Parts:
- gave numbers to parts that had none: 1
Changed lines of the file:
@@
 XBEE_TX
 $Comp
-L FSAE_Library:XBEE_Explorer U?
+L FSAE_Library:XBEE_Explorer U47
 U 1 1 5E6C9767
 P 8000 3000
-F 0 "U?" H 8528 2625 50  0000 L CNN
+F 0 "U47" H 8528 2625 50  0000 L CNN
 F 1 "XBEE_Explorer" H 8300 3250 50  0001 C CNN
 F 2 "" H 8500 3500 50  0001 C CNN
@@
 	7500 3000 7500 4000
 $Comp
-L FSAE_Library:GND #PWR?
+L FSAE_Library:GND #PWR022
 U 1 1 5E6D5A9D
 P 7500 4000
-F 0 "#PWR?" H 7500 3800 50  0001 C CNN
+F 0 "#PWR022" H 7500 3800 50  0001 C CNN
 F 1 "GND" H 7504 3846 50  0000 C CNN
 F 2 "" H 7500 3950 50  0001 C CNN
