File: Schematics/F20_Wiring_Diagrams/F20_ROOT_WIRING/F20_W_Engine_Sensors.sch (KiCad schematic (older format))
At the start: 22 parts

Commit message: Added engine side shifter wiring. Started engine side power management wiring
Parts:
- renumbered ICR7 to ICR1, ICR1 to ICR2, ICR2 to ICR3, ICR3 to ICR4, ICR4 to ICR5, ICR5 to ICR6, ICR6 to ICR7
Other:
- note added: "If reusing old injector/coil\nharnesses, there may be\ninterconnects here"
Changed lines of the file:
@@
 $Descr A 11000 8500
 encoding utf-8
-Sheet 2 2
-Title "Engine Sensors"
-Date "2020-06-20"
+Sheet 2 3
+Title "Engine Side - Sensors"
+Date "2020-06-22"
 Rev "A"
 Comp "F20"
@@
 12SI
 $Comp
-L FSAE_Library:DTM04-2P ICR2
+L FSAE_Library:DTM04-2P ICR3
 U 1 1 5EF0B53C
 P 7300 3000
-F 0 "ICR2" H 7050 3300 50  0000 R CNN
+F 0 "ICR3" H 7050 3300 50  0000 R CNN
 F 1 "DTM04-2P" H 7250 3200 50  0000 R CNN
 F 2 "" H 7300 3100 50  0001 C CNN
@@
 S3
 $Comp
-L FSAE_Library:DTM06-3P ICR3
+L FSAE_Library:DTM06-3P ICR4
 U 1 1 5EF4A6C4
 P 7400 2300
-F 0 "ICR3" H 7350 2600 50  0000 C CNN
+F 0 "ICR4" H 7350 2600 50  0000 C CNN
 F 1 "DTM06-3P" H 7458 2524 50  0000 C CNN
 F 2 "" H 7600 2400 50  0001 C CNN
@@
 7AG1
 $Comp
-L FSAE_Library:DTM04-2P ICR4
+L FSAE_Library:DTM04-2P ICR5
 U 1 1 5EFCA157
 P 8800 3000
-F 0 "ICR4" H 8550 3300 50  0000 R CNN
+F 0 "ICR5" H 8550 3300 50  0000 R CNN
 F 1 "DTM04-2P" H 8750 3200 50  0000 R CNN
 F 2 "" H 8800 3100 50  0001 C CNN
@@
 	9300 2500 9100 2500
 $Comp
-L FSAE_Library:DTM06-3P ICR5
+L FSAE_Library:DTM06-3P ICR6
 U 1 1 5EFCA164
 P 8900 2300
-F 0 "ICR5" H 8850 2600 50  0000 C CNN
+F 0 "ICR6" H 8850 2600 50  0000 C CNN
 F 1 "DTM06-3P" H 8958 2524 50  0000 C CNN
 F 2 "" H 9100 2400 50  0001 C CNN
@@
 	9600 1800 9400 1800
 $Comp
-L FSAE_Library:DTM06-3P ICR6
+L FSAE_Library:DTM06-3P ICR7
 U 1 1 5EFCF714
 P 9200 1600
-F 0 "ICR6" H 9150 1900 50  0000 C CNN
+F 0 "ICR7" H 9150 1900 50  0000 C CNN
 F 1 "DTM06-3P" H 9258 1824 50  0000 C CNN
 F 2 "" H 9400 1700 50  0001 C CNN
@@
 Fan
 $Comp
-L FSAE_Library:DTM04-2P ICR1
+L FSAE_Library:DTM04-2P ICR2
 U 1 1 5EEFFACE
 P 6300 5500
-F 0 "ICR1" H 6250 5650 50  0000 C CNN
+F 0 "ICR2" H 6250 5650 50  0000 C CNN
 F 1 "DTM04-2P" H 6158 5724 50  0001 C CNN
 F 2 "" H 6300 5600 50  0001 C CNN
@@
 	4100 6700 4300 6700
 $Comp
-L FSAE_Library:DTM04-2P ICR7
+L FSAE_Library:DTM04-2P ICR1
 U 1 1 5F13E690
 P 4300 6700
-F 0 "ICR7" H 4200 7000 50  0000 R CNN
+F 0 "ICR1" H 4200 7000 50  0000 R CNN
 F 1 "DTM04-2P" H 4200 6900 50  0000 R CNN
 F 2 "" H 4300 6800 50  0001 C CNN
@@
 Wire Wire Line
 	6800 1400 6600 1400
-Text Label 6600 900  0    39   ~ 0
-17SI1
 Text Label 6600 1000 0    39   ~ 0
 17SI2
@@
 Wire Notes Line
 	7350 850  7050 850
-Wire Bus Line
-	4000 6700 4000 7000
-Wire Bus Line
-	4000 7250 4000 7500
-Wire Bus Line
-	4350 1850 4350 3900
-Wire Bus Line
-	3100 4100 3100 5100
-Wire Bus Line
-	6500 900  6500 3900
-Wire Bus Line
-	2000 4000 2000 5150
-Wire Bus Line
-	4750 1850 4750 5150
-Wire Bus Line
-	2000 3050 2000 4000
-Wire Bus Line
-	2000 4000 9700 4000
 Text Notes 6400 3950 0    39   ~ 0
 6
+Text Notes 3500 3550 0    39   ~ 0
+If reusing old injector/coil\nharnesses, there may be\ninterconnects here
+Wire Notes Line
+	3450 3350 3450 3600
+Wire Notes Line
+	3450 3600 4850 3600
+Wire Notes Line
+	4850 3600 4850 3350
+Wire Notes Line
+	4850 3350 3450 3350
+Wire Bus Line
+	4000 6700 4000 7000
+Wire Bus Line
+	4000 7250 4000 7500
+Wire Bus Line
+	4350 1850 4350 3900
+Wire Bus Line
+	3100 4100 3100 5100
+Wire Bus Line
+	6500 900  6500 3900
+Wire Bus Line
+	2000 4000 2000 5150
+Wire Bus Line
+	4750 1850 4750 5150
+Wire Bus Line
+	2000 3050 2000 4000
+Wire Bus Line
+	2000 4000 9700 4000
+Text Label 6600 900  0    39   ~ 0
+17SI1
 $EndSCHEMATC
