File: Schematics/F20_Wiring_Diagrams/F20_ROOT_WIRING/F20_W_Eng_Sensors.sch (KiCad schematic (older format))
At the start: 22 parts

Commit message: Added shifter, brake light wiring, organized pwr mgmt diagrams
Parts:
- removed ICR2: DTM04-2P, symbol FSAE_Library:DTM04-2P
- added ICP3, ICP5, ICP6: DTM06-2S, symbol FSAE_Library:DTM06-2S
- added ICP4: DTM06-3S, symbol FSAE_Library:DTM06-3S
- added ICR10, ICR7, ICR9: DTM04-2P, symbol FSAE_Library:DTM04-2P
- added ICR8: DTM06-3P, symbol FSAE_Library:DTM06-3P
- added PT1, PT3, PT4: CompPigTail_2, symbol FSAE_Library:CompPigTail_2
- added PT2: CompPigTail_3, symbol FSAE_Library:CompPigTail_3
- renumbered ICR3 to ICR2, ICR4 to ICR3, ICR5 to ICR4, ICR6 to ICR5, ICR7 to ICR6
Connections:
- net 5BP: now also ICR7.1
- net 5CG: now also ICR7.2
- net 22SI: now reaches ICP1.21
- net 22SI: now also ICR10.1
- new net: ICP3.1, PT1.~
- new net: ICP3.2, PT1.~
- new net: ICP4.1, PT2.~
- new net: ICP4.2, PT2.~
- new net: ICP4.3, PT2.~
- new net: ICP5.1, PT3.~
- new net: ICP5.2, PT3.~
- new net: ICP6.1, PT4.~
- new net: ICP6.2, PT4.~
- new net 18CT: ICR8.2
- new net 19CT: ICR8.3
- new net 20CT: ICR9.2
- new net 21BP: ICR8.1, ICR9.1
- new net 22CG: ICR10.2
- no-connect marks 3 -> 2
Other:
- note added: "* Crank/Cam shielded harnesses,\nO2 sensor harness and the shifter\nharness pass directly through firewall"
- note added: "4"
- note added: "Brake\nLight"
- note added: "Clutch"
- note added: "Ground strategy\nflexible"
- note added: "S5"
- note added: "Up/Down\nShift"
- note removed: "CRANK/CAM shielded harnesses\nand O2 sensor harness pass\ndirectly through firewall"
- moved on the sheet: ICP2, ICR1
